File: ESP-WROOM-32-Breakout.brd (EAGLE design)
At the start: 89.5 x 38 mm, 76 parts, among them U3 ESP-WROOM-32

Commit message: Finished layout
Parts:
- removed AO3400: (no value), microbuilder:SOT23-R
- removed AO3401: (no value), microbuilder:SOT23-WIDE
- removed J10, J11, J12, J9: (no value), SparkFun-Connectors:1X03_NO_SILK
- removed J15, J16, J17: (no value), SparkFun-Connectors:1X06_NO_SILK
- removed J18, J19: (no value), SparkFun-Connectors:1X04_NO_SILK
- removed J24, J25: (no value), microbuilder:1X06_ROUND_70
- removed JP13: G, microbuilder:1X01_2MM
- removed JP14: D, microbuilder:1X01_2MM
- removed JP15: S, microbuilder:1X01_2MM
- removed JP16: D, pinhead:1X01
- removed JP17: G, pinhead:1X01
- removed JP18: S, pinhead:1X01
- removed R14, R15, R16, R17: 10k, rcl:R1206
- removed TPL2: TPL5111DDCR, TPL5111DDCR:SOT95P280X110-6N
- added J1: (no value), SparkFun-Connectors:USB-B-MICRO-SMD
- added JP1: (no value), microbuilder:1X03_ROUND_76
- added JP2, JP3, JP4, JP5: (no value), microbuilder:1X01_2MM
- added Q1: (no value), microbuilder:SOT23-WIDE
- moved R13 86.3 mm to (59.9, 27.1)
- moved R1 45.7 mm to (73.9, 26.4), turned to 180 degrees
- moved R11 44.9 mm to (63.8, 33.0), turned to 90 degrees
- moved C6 42.7 mm to (80.6, 35.6)
- moved R20 38.9 mm to (74.8, 35.7), turned to 0 degrees
- moved R3 37.9 mm to (68.6, 26.4), turned to 0 degrees
- moved U$1 35.8 mm to (80.6, 31.8), turned to 90 degrees
- moved C5 29.7 mm to (70.7, 34.0), turned to 90 degrees
- moved LED2 29.3 mm to (74.9, 32.6), turned to 90 degrees
- moved R19 24.0 mm to (72.6, 29.8), turned to 180 degrees
- moved C1 20.4 mm to (32.4, 14.1), turned to 180 degrees
- moved R2 17.2 mm to (38.6, 14.1), turned to 180 degrees
- moved C2 7.81 mm to (38.5, 17.3)
- moved C3 7.45 mm to (40.1, 22.5)
- moved R12 5.41 mm to (47.0, 15.2)
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Connections:
- removed net N$14: AO3400.1, JP17.1
- removed net N$16: AO3400.3, JP16.1
- removed net N$17: AO3400.2, JP18.1
- removed net N$32: J9.3
- removed net N$33: J9.2
- removed net N$35: J9.1
- removed net N$39: J12.1, TPL2.3
- removed net N$40: J11.1, TPL2.4
- removed net N$41: J11.3, TPL2.6
- removed net N$42: J10.1
- removed net N$43: J10.3
- removed net N$55: J25.6, R11.1
- removed net N$56: J24.1, R11.2
- removed net N$57: J24.2, R13.2
- removed net N$58: J24.3, R14.2
- removed net N$59: J24.4, R15.2
- removed net N$60: J24.5, R16.2
- removed net N$61: J24.6, R17.2
- removed net N$62: J25.1, R17.1
- removed net N$63: J25.2, R16.1
- removed net N$64: J25.3, R15.1
- removed net N$65: J25.4, R14.1
- removed net N$66: J25.5, R13.1
- net +5V: now also J1.VBUS
- net GND: now also J1.GND
- net IO16: now also SPI.8; no longer SPI.7
- net IO17: now also SPI.7; no longer SPI.8
- net IO25: now also IN/OUT.2; no longer IN/OUT.6
- net IO26: now also IN/OUT.1; no longer IN/OUT.7
- net IO32: now also IN/OUT.4; no longer IN/OUT.5
- net IO33: now also IN/OUT.3; no longer IN/OUT.4
- net IO34: now also IN/OUT.6; no longer IN/OUT.3
- net IO35: now also IN/OUT.5; no longer IN/OUT.2
- net IO39: now also IN/OUT.7; no longer IN/OUT.1
- net N$11: now also JP3.1, R11.1; no longer J12.3, TPL2.1
- net N$12: now also JP4.1, R13.2; no longer J12.2, TPL2.2
- net N$13: now also JP5.1, R13.1; no longer AO3401.3, JP15.1
- net N$2: now also JP1.1, Q1.2; no longer AO3401.2, JP14.1
- net N$6: now also JP1.2, Q1.1; no longer AO3401.1, JP13.1
- net N$7: now also JP1.3, Q1.3; no longer J10.2
- net N$9: now also JP2.1, R11.2; no longer J11.2, TPL2.5
Routing:
- net GND: track 26.5 -> 244.0 mm
- net +3V3: track 26.5 -> 181.5 mm, vias 0 -> 5
- net VDD: track 0.00 -> 85.4 mm
- net SCL: track 0.00 -> 72.7 mm, vias 0 -> 2
- net +5V: track 0.00 -> 72.3 mm, vias 0 -> 1
- net SDA: track 0.00 -> 71.9 mm, vias 0 -> 2
- net TXD0: track 0.00 -> 70.4 mm, vias 0 -> 2
- net IO36: track 0.00 -> 67.3 mm, vias 0 -> 2
- net BAT: track 0.00 -> 55.7 mm, vias 0 -> 1
- net IO27: track 0.00 -> 46.9 mm, vias 0 -> 2
- net IO14: track 0.00 -> 40.3 mm, vias 0 -> 2
- net N$4: track 0.00 -> 39.8 mm
- net RXD0: track 0.00 -> 37.3 mm, vias 0 -> 3
- net IO0: track 0.00 -> 35.3 mm, vias 0 -> 2
- net EN: track 0.00 -> 30.6 mm, vias 0 -> 1
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Other:
- board text added: "v.2 March 2019"
- board text removed: "Jan 2019"

Commit message: save
Parts:
- removed POWER_IN: (no value), SparkFun-Connectors:1X03_NO_SILK
- added +5V, BAT: (no value), SparkFun-Connectors:1X02
- added C7, C8, C9: 100nF, microbuilder:1206
Connections:
- removed net N$67: R20.2, U$1.5
- new net N$32: R20.1, U$1.5
- net +3V3: now also C7.1, C8.2
- net +5V: now also +5V.2, C5.2, S3.1; no longer C5.1, POWER_IN.3, S3.3
- net BAT: now also BAT.2, C6.1, C9.1, S3.3; no longer C6.2, POWER_IN.1, S3.1
- net GND: now also +5V.1, BAT.1, C5.1, C6.2, C7.2, C8.1, C9.2, R20.2; no longer C5.2, C6.1, POWER_IN.2, R20.1
Routing:
- net BAT: track 55.7 -> 0.00 mm, vias 1 -> 0
- net GND: track 244.0 -> 215.4 mm
- net N$16: track 24.7 -> 0.00 mm
- net +5V: track 72.3 -> 51.9 mm
- net N$67: track 6.42 -> 0.00 mm, vias 2 -> 0
- net VDD: track 85.4 -> 79.6 mm
