File: ESP-WROOM-32-Breakout.sch (EAGLE design)
At the start: 76 parts, among them U3 ESP-WROOM-32

Commit message: Finished layout
Parts:
- removed AO3400: (no value), microbuilder:MOSFET-NREFLOW
- removed AO3401: (no value), microbuilder:MOSFET-PWIDE
- removed J10, J11, J12, J9: (no value), SparkFun-Connectors:CONN_031X03_NO_SILK
- removed J15, J16, J17: (no value), SparkFun-Connectors:CONN_06NO_SILK_NO_POP
- removed J18, J19: (no value), SparkFun-Connectors:CONN_041X04_NO_SILK
- removed J24, J25: (no value), microbuilder:HEADER-1X670MIL
- removed JP13: G, microbuilder:HEADER-1X12MM
- removed JP14: D, microbuilder:HEADER-1X12MM
- removed JP15: S, microbuilder:HEADER-1X12MM
- removed JP16: D, pinhead:PINHD-1X1
- removed JP17: G, pinhead:PINHD-1X1
- removed JP18: S, pinhead:PINHD-1X1
- removed R14, R15, R16, R17: 10k, rcl:R-EU_R1206
- removed TPL2: TPL5111DDCR, TPL5111DDCR:TPL5111DDCR
- added J1: (no value), SparkFun-Connectors:USB_MICRO-B_FEMALE-SMT
- added JP1: (no value), microbuilder:HEADER-1X376MIL
- added JP2, JP3, JP4, JP5: (no value), microbuilder:HEADER-1X12MM
- added Q1: (no value), microbuilder:MOSFET-NWIDE
Connections:
- removed net N$14: AO3400.G, JP17.1
- removed net N$16: AO3400.D, JP16.1
- removed net N$17: AO3400.S, JP18.1
- removed net N$32: J9.3
- removed net N$33: J9.2
- removed net N$35: J9.1
- removed net N$39: J12.1, TPL2.DELAY/M_DRV
- removed net N$40: J11.1, TPL2.DONE
- removed net N$41: J11.3, TPL2.EN/ONE_SHOT
- removed net N$42: J10.1
- removed net N$43: J10.3
- removed net N$55: J25.6, R11.1
- removed net N$56: J24.1, R11.2
- removed net N$57: J24.2, R13.2
- removed net N$58: J24.3, R14.2
- removed net N$59: J24.4, R15.2
- removed net N$60: J24.5, R16.2
- removed net N$61: J24.6, R17.2
- removed net N$62: J25.1, R17.1
- removed net N$63: J25.2, R16.1
- removed net N$64: J25.3, R15.1
- removed net N$65: J25.4, R14.1
- removed net N$66: J25.5, R13.1
- net +5V: now also J1.VBUS
- net GND: now also J1.GND
- net IO16: now also SPI.8; no longer SPI.7
- net IO17: now also SPI.7; no longer SPI.8
- net IO25: now also IN/OUT.2; no longer IN/OUT.6
- net IO26: now also IN/OUT.1; no longer IN/OUT.7
- net IO32: now also IN/OUT.4; no longer IN/OUT.5
- net IO33: now also IN/OUT.3; no longer IN/OUT.4
- net IO34: now also IN/OUT.6; no longer IN/OUT.3
- net IO35: now also IN/OUT.5; no longer IN/OUT.2
- net IO39: now also IN/OUT.7; no longer IN/OUT.1
- net N$11: now also JP3.1, R11.1; no longer J12.3, TPL2.VDD
- net N$12: now also JP4.1, R13.2; no longer J12.2, TPL2.GND
- net N$13: now also JP5.1, R13.1; no longer AO3401.D, JP15.1
- net N$2: now also JP1.1, Q1.S; no longer AO3401.S, JP14.1
- net N$6: now also JP1.2, Q1.G; no longer AO3401.G, JP13.1
- net N$7: now also JP1.3, Q1.D; no longer J10.2
- net N$9: now also JP2.1, R11.2; no longer J11.2, TPL2.DRVN
Other:
- moved on the sheet: C6, POWER_IN, R19, S3

Commit message: save
Parts:
- removed POWER_IN: (no value), SparkFun-Connectors:CONN_031X03_NO_SILK
- added +5V, BAT: (no value), SparkFun-Connectors:CONN_02
- added C7, C8, C9: 100nF, microbuilder:CAP_CERAMIC1206
Connections:
- removed net N$67: R20.2, U$1.PROG
- new net N$32: R20.1, U$1.PROG
- net +3V3: now also C7.P$1, C8.P$2
- net +5V: now also +5V.2, C5.P$2, S3.O; no longer C5.P$1, POWER_IN.3, S3.S
- net BAT: now also BAT.2, C6.P$1, C9.P$1, S3.S; no longer C6.P$2, POWER_IN.1, S3.O
- net GND: now also +5V.1, BAT.1, C5.P$1, C6.P$2, C7.P$2, C8.P$1, C9.P$2, R20.2; no longer C5.P$2, C6.P$1, POWER_IN.2, R20.1
Other:
- moved on the sheet: 3400, 3401, C1, C2, C3, C4, C5, C6, I2C, IN/OUT, J13, J14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
